File: SchematicAndBoards/Devices/Switch-220v-HiLink-CC1101-AS07/Switch-220v-HiLink-CC1101-AS07.brd (EAGLE design)
At the start: 34 x 30.5 mm, 22 parts, among them T1 BTA12-600C

Commit message: Update schematic and boards
Parts:
- renumbered U$1 to U1
Other:
- board text added: "GND"
- board text added: "NRTS"
- board text added: "SWCLK"
- board text added: "SWDIO"
- board text added: "U_TX"
- board text added: "VDD3.3"
- board text added: "ver 0.5 alexsam@saewave.com"
